Commit message: fix: 完善机器人接入接口与 RGL 生命周期处理
统一挂载宏、桥接和实例配置的话题规则，支持自定义点云、IMU 与时钟源；扫描布局由依赖锁文件统一驱动，直接 Xacro 与 launch 均校验配置。

初始化失败立即停用并清理所有图分量；实体删除清理延后到串行 PreUpdate，修复并发释放导致的后端错误。增加独立父机器人构建、复位及删除重建回归。

补全 README 接入示例、变更记录及技术/正式发行检查。验证：101 项 Python 测试、35 个无 GPU 初始化故障点、原生 GPU 全套回归、无 GPU 容器构建及容器 GPU 接入生命周期测试通过；分发审查仍明确待确认。

File: urdf/demo.urdf.xacro (robot description, xacro)
@@ -5,6 +5,6 @@
   <xacro:arg name="xyz" default="0 0 1"/>
   <xacro:arg name="rpy" default="0 0 0"/>
-  <xacro:arg name="points_topic" default="/livox/mid360/points"/>
-  <xacro:arg name="imu_topic" default="/livox/mid360/imu"/>
+  <xacro:arg name="points_topic" default=""/>
+  <xacro:arg name="imu_topic" default=""/>
   <xacro:arg name="visual_mesh" default=""/>
   <xacro:arg name="mesh_rpy" default="0 0 0"/>

File: urdf/livox.xacro (robot description, xacro)
@@ -2,6 +2,26 @@
 <robot xmlns:xacro="http://www.ros.org/wiki/xacro">
   <!-- Reusable mount macro: parent owns world, robot_state_publisher and namespaces. -->
-  <xacro:macro name="livox_lidar" params="parent name:=mid360 model:=mid360 xyz:='0 0 0' rpy:='0 0 0' points_topic:=/livox/mid360/points imu_topic:=/livox/mid360/imu visual_mesh:='' mesh_rpy:='0 0 0'">
+  <xacro:include filename="$(find livox_lidar_simulation_gz)/urdf/validation.xacro"/>
+  <xacro:macro name="livox_lidar" params="parent name:=mid360 model:=mid360 xyz:='0 0 0' rpy:='0 0 0' points_topic:='' imu_topic:='' visual_mesh:='' mesh_rpy:='0 0 0' namespace:=livox">
+    <xacro:livox_require condition="${model in ['mid360', 'avia']}" message="Unsupported Livox model"/>
     <xacro:property name="cfg" value="${xacro.load_yaml('$(find livox_lidar_simulation_gz)/config/models/' + model + '.yaml')}"/>
+    <xacro:property name="preset" value="${xacro.load_yaml('$(find livox_lidar_simulation_gz)/dependencies/lock.json')['scan_presets'][model]}"/>
+    <xacro:property name="pattern_root" value="$(optenv RGL_PATTERNS_DIR)"/>
+    <xacro:property name="default_pattern_root" value="$(find livox_lidar_simulation_gz)/patterns"/>
+    <xacro:livox_validate_config cfg="${cfg}" preset="${preset}" model="${model}"/>
+    <xacro:livox_check_name value="${name}" first_letter="${True}"/>
+    <xacro:livox_require condition="${python.isinstance(namespace,str)}" message="namespace must be a string"/>
+    <xacro:if value="${namespace.strip('/') != ''}">
+      <xacro:livox_check_segments values="${namespace.strip('/').split('/')}"/>
+    </xacro:if>
+    <xacro:property name="topic_root" value="${'/' + '/'.join(v for v in [namespace.strip('/'), name] if v)}"/>
+    <xacro:property name="actual_points_topic" value="${points_topic or topic_root + '/points'}"/>
+    <xacro:property name="actual_imu_topic" value="${imu_topic or topic_root + '/imu'}"/>
+    <xacro:livox_check_topic value="${actual_points_topic}"/>
+    <xacro:livox_check_topic value="${actual_imu_topic}"/>
+    <xacro:livox_require condition="${actual_points_topic != actual_imu_topic}" message="Point cloud and IMU topics must differ"/>
+    <xacro:livox_check_vector value="${xyz}" field="xyz"/>
+    <xacro:livox_check_vector value="${rpy}" field="rpy"/>
+    <xacro:livox_check_vector value="${mesh_rpy}" field="mesh_rpy"/>
     <xacro:property name="sx" value="${cfg['size_x']}"/>
     <xacro:property name="sy" value="${cfg['size_y']}"/>
@@ -84,6 +104,6 @@
           <update_rate>${cfg['lidar_rate']}</update_rate>
           <update_on_paused_sim>false</update_on_paused_sim>
-          <topic>${points_topic}</topic><frame>${name}_lidar</frame>
-          <pattern_preset>${cfg['pattern']}</pattern_preset>
+          <topic>${actual_points_topic}</topic><frame>${name}_lidar</frame>
+          <pattern_preset_path pattern_count="${preset['pattern_groups']}" rays_per_frame="${preset['rays_per_frame']}">${pattern_root or default_pattern_root}/${preset['pattern_file']}</pattern_preset_path>
         </plugin>
       </sensor>
@@ -92,5 +112,5 @@
       <sensor name="${name}_imu_sensor" type="imu">
         <always_on>true</always_on><update_rate>${cfg['imu_rate']}</update_rate>
-        <topic>${imu_topic}</topic><gz_frame_id>${name}_imu</gz_frame_id>
+        <topic>${actual_imu_topic}</topic><gz_frame_id>${name}_imu</gz_frame_id>
       </sensor>
     </gazebo>

File: urdf/moving.urdf.xacro (robot description, xacro)
@@ -3,6 +3,6 @@
   <xacro:arg name="model" default="mid360"/><xacro:arg name="name" default="mid360"/>
   <xacro:arg name="xyz" default="0 0 1"/><xacro:arg name="rpy" default="0 0 0"/>
-  <xacro:arg name="points_topic" default="/livox/mid360/points"/>
-  <xacro:arg name="imu_topic" default="/livox/mid360/imu"/>
+  <xacro:arg name="points_topic" default=""/>
+  <xacro:arg name="imu_topic" default=""/>
   <xacro:arg name="visual_mesh" default=""/><xacro:arg name="mesh_rpy" default="0 0 0"/>
   <xacro:arg name="linear_velocity" default="0.1"/><xacro:arg name="angular_velocity" default="0.15"/>
