Commit message: feat(mid360): 接入精细彩色模型与官方名义外参

File: urdf/livox.xacro (robot description, xacro)
@@ -7,4 +7,5 @@
     <xacro:property name="sy" value="${cfg['size_y']}"/>
     <xacro:property name="sz" value="${cfg['size_z']}"/>
+    <xacro:property name="actual_mesh" value="${cfg['visual_mesh'] if visual_mesh == '' else ('' if visual_mesh == 'primitive' else visual_mesh)}"/>
     <!-- Tiny numerical frame masses keep fixed sensor links in Gazebo's URDF conversion. -->
     <xacro:property name="frame_mass" value="0.000001"/>
@@ -17,6 +18,11 @@
       </inertial>
       <collision name="${name}_collision">
-        <origin xyz="0 0 ${sz / 2}"/>
-        <geometry><box size="${sx} ${sy} ${sz}"/></geometry>
+        <origin xyz="0 0 ${cfg['collision_body_height'] / 2}"/>
+        <geometry><box size="${sx} ${sy} ${cfg['collision_body_height']}"/></geometry>
+      </collision>
+      <!-- Approximate connector envelope: manual width including connector is 73 mm. -->
+      <collision name="${name}_connector_collision">
+        <origin xyz="-0.0365 0 0.0143" rpy="0 1.5707963267948966 0"/>
+        <geometry><cylinder radius="0.0062" length="0.008"/></geometry>
       </collision>
     </link>
@@ -28,11 +34,11 @@
       <inertial><mass value="${frame_mass}"/><inertia ixx="1e-9" iyy="1e-9" izz="1e-9" ixy="0" ixz="0" iyz="0"/></inertial>
       <!-- RGL excludes visuals in the sensor's own link, not the whole robot. -->
-      <xacro:if value="${visual_mesh != ''}">
+      <xacro:if value="${actual_mesh != ''}">
         <visual name="${name}_external_mesh">
           <origin xyz="0 0 ${-cfg['measurement_z']}" rpy="${mesh_rpy}"/>
-          <geometry><mesh filename="${visual_mesh}"/></geometry>
+          <geometry><mesh filename="${actual_mesh}"/></geometry>
         </visual>
       </xacro:if>
-      <xacro:unless value="${visual_mesh != ''}">
+      <xacro:unless value="${actual_mesh != ''}">
         <visual name="${name}_base_visual">
           <origin xyz="0 0 ${sz * 0.28 - cfg['measurement_z']}"/>
@@ -56,5 +62,5 @@
     <joint name="${name}_imu_joint" type="fixed">
       <parent link="${name}_body"/><child link="${name}_imu"/>
-      <origin xyz="0 0 ${cfg['imu_z']}"/>
+      <origin xyz="${cfg['imu_xyz'][0]} ${cfg['imu_xyz'][1]} ${cfg['imu_xyz'][2]}"/>
     </joint>
     <gazebo reference="${name}_lidar_joint"><preserveFixedJoint>true</preserveFixedJoint></gazebo>

Commit message: feat: 完善首版移动验证、多型号预览与交付工具

File: urdf/livox.xacro (robot description, xacro)
@@ -22,8 +22,10 @@
       </collision>
       <!-- Approximate connector envelope: manual width including connector is 73 mm. -->
+      <xacro:if value="${cfg['connector_collision']}">
       <collision name="${name}_connector_collision">
         <origin xyz="-0.0365 0 0.0143" rpy="0 1.5707963267948966 0"/>
         <geometry><cylinder radius="0.0062" length="0.008"/></geometry>
       </collision>
+      </xacro:if>
     </link>
     <joint name="${name}_mount" type="fixed">
@@ -41,4 +43,5 @@
       </xacro:if>
       <xacro:unless value="${actual_mesh != ''}">
+        <xacro:if value="${cfg['visual_style'] == 'dome'}">
         <visual name="${name}_base_visual">
           <origin xyz="0 0 ${sz * 0.28 - cfg['measurement_z']}"/>
@@ -51,4 +54,17 @@
           <material name="${name}_blue"><color rgba="0.05 0.23 0.3 1"/></material>
         </visual>
+        </xacro:if>
+        <xacro:if value="${cfg['visual_style'] == 'front_window'}">
+          <visual name="${name}_housing">
+            <origin xyz="0 0 ${sz/2-cfg['measurement_z']}"/>
+            <geometry><box size="${sx} ${sy} ${sz}"/></geometry>
+            <material name="${name}_silver"><color rgba="0.65 0.68 0.72 1"/></material>
+          </visual>
+          <visual name="${name}_window">
+            <origin xyz="${sx/2+0.0001} 0 ${sz/2-cfg['measurement_z']}"/>
+            <geometry><box size="0.0001 ${sy*.85} ${sz*.7}"/></geometry>
+            <material name="${name}_window_black"><color rgba="0.02 0.025 0.035 1"/></material>
+          </visual>
+        </xacro:if>
       </xacro:unless>
     </link>

Commit message: chore: 清理开发过程文件并整理 Avia 运行资产
移出模型制作源和工具，删除历史计划、迁移基线与一次性交付报告。精简用户文档和几何报告，明确安装资源清单，保留来源与分发限制。

纳入 Avia 精细模型、型号碰撞配置及回归测试；保留依赖锁定。验证：47 项单元测试、元信息检查及差异检查通过；清理后已验证独立构建、单实例、混合双实例和两型号移动复位。

File: urdf/livox.xacro (robot description, xacro)
@@ -7,5 +7,5 @@
     <xacro:property name="sy" value="${cfg['size_y']}"/>
     <xacro:property name="sz" value="${cfg['size_z']}"/>
-    <xacro:property name="actual_mesh" value="${cfg['visual_mesh'] if visual_mesh == '' else ('' if visual_mesh == 'primitive' else visual_mesh)}"/>
+    <xacro:property name="actual_mesh" value="${xacro.fatal('Avia primitive appearance has been removed; use the detailed mesh') if model == 'avia' and visual_mesh == 'primitive' else (cfg['visual_mesh'] if visual_mesh == '' else ('' if visual_mesh == 'primitive' else visual_mesh))}"/>
     <!-- Tiny numerical frame masses keep fixed sensor links in Gazebo's URDF conversion. -->
     <xacro:property name="frame_mass" value="0.000001"/>
@@ -21,9 +21,16 @@
         <geometry><box size="${sx} ${sy} ${cfg['collision_body_height']}"/></geometry>
       </collision>
-      <!-- Approximate connector envelope: manual width including connector is 73 mm. -->
+      <!-- Lightweight, model-specific connector envelope; never use CAD for collision. -->
       <xacro:if value="${cfg['connector_collision']}">
       <collision name="${name}_connector_collision">
-        <origin xyz="-0.0365 0 0.0143" rpy="0 1.5707963267948966 0"/>
-        <geometry><cylinder radius="0.0062" length="0.008"/></geometry>
+        <origin xyz="${cfg['connector']['xyz']}" rpy="${cfg['connector']['rpy']}"/>
+        <geometry>
+          <xacro:if value="${cfg['connector']['shape'] == 'cylinder'}">
+            <cylinder radius="${cfg['connector']['radius']}" length="${cfg['connector']['length']}"/>
+          </xacro:if>
+          <xacro:if value="${cfg['connector']['shape'] == 'box'}">
+            <box size="${cfg['connector']['size']}"/>
+          </xacro:if>
+        </geometry>
       </collision>
       </xacro:if>
@@ -54,16 +61,4 @@
           <material name="${name}_blue"><color rgba="0.05 0.23 0.3 1"/></material>
         </visual>
-        </xacro:if>
-        <xacro:if value="${cfg['visual_style'] == 'front_window'}">
-          <visual name="${name}_housing">
-            <origin xyz="0 0 ${sz/2-cfg['measurement_z']}"/>
-            <geometry><box size="${sx} ${sy} ${sz}"/></geometry>
-            <material name="${name}_silver"><color rgba="0.65 0.68 0.72 1"/></material>
-          </visual>
-          <visual name="${name}_window">
-            <origin xyz="${sx/2+0.0001} 0 ${sz/2-cfg['measurement_z']}"/>
-            <geometry><box size="0.0001 ${sy*.85} ${sz*.7}"/></geometry>
-            <material name="${name}_window_black"><color rgba="0.02 0.025 0.035 1"/></material>
-          </visual>
         </xacro:if>
       </xacro:unless>

Commit message: fix(avia): 修正传感器坐标并完善仿真验证
按官方手册设置 IMU 相对位移，将雷达原点配准到 CAD 前窗；使用完整 measurement_xyz 并保留模型安装位置。近端保守截断改为 1 m，按型号尺寸调整 RViz 近景。

补充扫描视场、量程、空点云、遮挡及实际渲染测试，同步中英文 README 与来源说明。验证：104 项 Python 测试通过，GPU 回归、DAE/GLB 可视检查及 Avia 600 秒稳定性测试通过。分发条件仍保留待确认状态。

File: urdf/livox.xacro (robot description, xacro)
@@ -65,5 +65,5 @@
       <xacro:if value="${actual_mesh != ''}">
         <visual name="${name}_external_mesh">
-          <origin xyz="0 0 ${-cfg['measurement_z']}" rpy="${mesh_rpy}"/>
+          <origin xyz="${-cfg['measurement_xyz'][0]} ${-cfg['measurement_xyz'][1]} ${-cfg['measurement_xyz'][2]}" rpy="${mesh_rpy}"/>
           <geometry><mesh filename="${actual_mesh}"/></geometry>
         </visual>
@@ -72,10 +72,10 @@
         <xacro:if value="${cfg['visual_style'] == 'dome'}">
         <visual name="${name}_base_visual">
-          <origin xyz="0 0 ${sz * 0.28 - cfg['measurement_z']}"/>
+          <origin xyz="${-cfg['measurement_xyz'][0]} ${-cfg['measurement_xyz'][1]} ${sz * 0.28 - cfg['measurement_xyz'][2]}"/>
           <geometry><box size="${sx} ${sy} ${sz * 0.56}"/></geometry>
           <material name="${name}_silver"><color rgba="0.65 0.68 0.72 1"/></material>
         </visual>
         <visual name="${name}_cover_visual">
-          <origin xyz="0 0 ${sz * 0.76 - cfg['measurement_z']}"/>
+          <origin xyz="${-cfg['measurement_xyz'][0]} ${-cfg['measurement_xyz'][1]} ${sz * 0.76 - cfg['measurement_xyz'][2]}"/>
           <geometry><cylinder radius="${sx * 0.44}" length="${sz * 0.48}"/></geometry>
           <material name="${name}_blue"><color rgba="0.05 0.23 0.3 1"/></material>
@@ -86,5 +86,5 @@
     <joint name="${name}_lidar_joint" type="fixed">
       <parent link="${name}_body"/><child link="${name}_lidar"/>
-      <origin xyz="0 0 ${cfg['measurement_z']}"/>
+      <origin xyz="${cfg['measurement_xyz'][0]} ${cfg['measurement_xyz'][1]} ${cfg['measurement_xyz'][2]}"/>
     </joint>
     <link name="${name}_imu">

File: urdf/validation.xacro (robot description, xacro)
@@ -40,10 +40,12 @@
     <xacro:livox_require condition="${python.type(preset['pattern_groups']) == int and preset['pattern_groups'] > 0 and python.type(preset['rays_per_frame']) == int and preset['rays_per_frame'] > 0}" message="Scan layout requires positive integers"/>
     <xacro:livox_require condition="${'/' not in preset['pattern_file'] and '..' not in preset['pattern_file']}" message="Invalid pattern filename"/>
-    <xacro:livox_check_fields cfg="${cfg}" fields="${['lidar_rate','imu_rate','mass','size_x','size_y','size_z','collision_body_height','measurement_z','range_max']}"/>
+    <xacro:livox_check_fields cfg="${cfg}" fields="${['lidar_rate','imu_rate','mass','size_x','size_y','size_z','collision_body_height','range_max']}"/>
     <xacro:livox_check_number value="${cfg['range_min']}" field="range_min"/>
-    <xacro:livox_require condition="${0 &lt;= cfg['range_min'] &lt; cfg['range_max'] and cfg['measurement_z'] &lt;= cfg['size_z'] and cfg['mass'] > 0.000002 and cfg['lidar_rate'] &lt;= 1000000 and cfg['imu_rate'] &lt;= 1000000}" message="Invalid range, origin, mass or update rate"/>
+    <xacro:livox_require condition="${0 &lt;= cfg['range_min'] &lt; cfg['range_max'] and cfg['mass'] > 0.000002 and cfg['lidar_rate'] &lt;= 1000000 and cfg['imu_rate'] &lt;= 1000000}" message="Invalid range, mass or update rate"/>
+    <xacro:livox_check_vector value="${cfg['measurement_xyz']}" field="measurement_xyz"/>
+    <xacro:livox_require condition="${python.abs(cfg['measurement_xyz'][0]) &lt;= cfg['size_x']/2 and python.abs(cfg['measurement_xyz'][1]) &lt;= cfg['size_y']/2 and 0 &lt; cfg['measurement_xyz'][2] &lt;= cfg['size_z']}" message="Invalid measurement origin"/>
     <xacro:livox_check_vector value="${cfg['imu_xyz']}" field="imu_xyz"/>
     <xacro:livox_check_vector value="${cfg['imu_from_lidar_xyz']}" field="imu_from_lidar_xyz"/>
-    <xacro:livox_require condition="${python.all(math.isclose(a,b,abs_tol=1e-8) for a,b in python.zip(cfg['imu_from_lidar_xyz'],[cfg['imu_xyz'][0],cfg['imu_xyz'][1],cfg['imu_xyz'][2]-cfg['measurement_z']]))}" message="IMU offsets disagree with measurement origin"/>
+    <xacro:livox_require condition="${python.all(math.isclose(a,b-c,abs_tol=1e-8) for a,b,c in python.zip(cfg['imu_from_lidar_xyz'],cfg['imu_xyz'],cfg['measurement_xyz']))}" message="IMU offsets disagree with measurement origin"/>
     <xacro:livox_require condition="${python.type(cfg['connector_collision']) == bool}" message="connector_collision must be boolean"/>
     <xacro:if value="${cfg['connector_collision']}">
